File: 0036_LORA_Module_E32-433T30D.kicad_sch (KiCad schematic)
At the start: 12 parts, among them J1 Conn_01x07_Pin, Q1 MMBT3906, Q2 3906, Q3 MMBT3906

Commit message: Add files via upload
Parts:
- removed D3: LED, symbol Device:LED
- removed Q3: MMBT3906, Package_TO_SOT_SMD:SOT-23, symbol Transistor_BJT:MMBT3906
- removed R3: R, symbol Device:R
- removed S1: DS01, DS01254S02BE, symbol DS01-254-S-02BE:DS01-254-S-02BE
- added D4: LED, LED_SMD:LED_0805_2012Metric, symbol Device:LED
- added R4, R5: 0r, Resistor_SMD:R_0805_2012Metric, symbol Device:R
- added R7: R, Resistor_SMD:R_0805_2012Metric, symbol Device:R
- added U1: ~, Moduler_:pin_header_5-3, symbol moduler_pin:air
- C1: footprint (none) -> Capacitor_SMD:C_0805_2012Metric
- D1, D2: footprint (none) -> LED_SMD:LED_0805_2012Metric
- J1: footprint (none) -> Connector_PinHeader_2.54mm:PinHeader_1x07_P2.54mm_Vertical
- R1, R2: footprint (none) -> Resistor_SMD:R_0805_2012Metric
Connections:
- net GND: now also J1.7 (GND), D4.1 (K), U1.9; no longer J1.GND
- net RX: now also J1.3 (RX), R5.2, U1.11; no longer J1.TX, Q1.1 (B)
- net TX: now also J1.4 (TX), R4.2, U1.10; no longer J1.RX, Q2.1 (B)
- net VCC renamed +3V3
- net +3V3: now also J1.6 (VCC), R7.2, U1.8; no longer J1.VCC
- new net: Q2.1 (B), R5.1
- new net: Q1.1 (B), R4.1
- new net: D4.2 (A), R7.1
- new net AUX: J1.5 (AUX), U1.14
- new net M1: J1.2 (M1), U1.12
- new net M2: J1.1 (M0), U1.13
- no-connect marks 0 -> 11
Other:
- note added: "AIR PIN"
- note added: "LORA"
- moved on the sheet: C1, D1, D2, Q2, R1, R2
